File: decimator_pcb.kicad_pcb (KiCad board)
At the start: 2 copper layers, 149 x 115.5 mm, 58 parts

Commit message: x glyph
Parts:
- added G***: LOGO, Library:x, F.Cu at (135.0, 136.0)
Changed lines of the file:
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@@
     )
+  )
+  (footprint "Library:x" (layer "F.Cu")
+    (at 135 136)
+    (attr board_only exclude_from_pos_files exclude_from_bom)
+    (fp_text reference "G***" (at 0 0) (layer "F.SilkS") hide
+      (effects (font (size 1.524 1.524) (thickness 0.3)))
+    )
+    (fp_text value "LOGO" (at 0.75 0) (layer "F.SilkS") hide
+      (effects (font (size 1.524 1.524) (thickness 0.3)))
+    )
+    (fp_poly (pts
+        (xy -0.375024 -1.000062)
+        (xy -0.125008 -1.000062)
+        (xy -0.125008 -0.750047)
+        (xy 0 -0.750047)
+        (xy 0 -0.625039)
+        (xy 0.125007 -0.625039)
+        (xy 0.125007 -0.750047)
+        (xy 0.250015 -0.750047)
+        (xy 0.250015 -0.875054)
+        (xy 0.375023 -0.875054)
+        (xy 0.375023 -1.000062)
+        (xy 0.875053 -1.000062)
+        (xy 0.875053 -0.875054)
+        (xy 1.000061 -0.875054)
+        (xy 1.000061 -0.375024)
+        (xy 0.750046 -0.375024)
+        (xy 0.750046 -0.750047)
+        (xy 0.50003 -0.750047)
+        (xy 0.50003 -0.625039)
+        (xy 0.375023 -0.625039)
+        (xy 0.375023 -0.500031)
+        (xy 0.250015 -0.500031)
+        (xy 0.250015 -0.375024)
+        (xy 0.125007 -0.375024)
+        (xy 0.125007 0)
+        (xy 0 0)
+        (xy 0 0.250015)
+        (xy 0.125007 0.250015)
+        (xy 0.125007 0.50003)
+        (xy 0.250015 0.50003)
+        (xy 0.250015 0.625038)
+        (xy 0.50003 0.625038)
+        (xy 0.50003 0.50003)
+        (xy 0.625038 0.50003)
+        (xy 0.625038 0.375023)
+        (xy 0.750046 0.375023)
+        (xy 0.750046 0.250015)
+        (xy 0.875053 0.250015)
+        (xy 0.875053 0.50003)
+        (xy 0.750046 0.50003)
+        (xy 0.750046 0.625038)
+        (xy 0.625038 0.625038)
+        (xy 0.625038 0.750046)
+        (xy 0.50003 0.750046)
+        (xy 0.50003 0.875053)
+        (xy 0.125007 0.875053)
+        (xy 0.125007 0.750046)
+        (xy 0 0.750046)
+        (xy 0 0.625038)
+        (xy -0.125008 0.625038)
+        (xy -0.125008 0.375023)
+        (xy -0.250016 0.375023)
+        (xy -0.250016 0.50003)
+        (xy -0.375024 0.50003)
+        (xy -0.375024 0.625038)
+        (xy -0.500031 0.625038)
+        (xy -0.500031 0.750046)
+        (xy -0.625039 0.750046)
+        (xy -0.625039 0.875053)
+        (xy -1.12507 0.875053)
+        (xy -1.12507 0.750046)
+        (xy -1.250077 0.750046)
+        (xy -1.250077 0.50003)
+        (xy -1.12507 0.50003)
+        (xy -1.12507 0.375023)
+        (xy -0.875054 0.375023)
+        (xy -0.875054 0.50003)
+        (xy -0.625039 0.50003)
+        (xy -0.625039 0.375023)
+        (xy -0.500031 0.375023)
+        (xy -0.500031 0.250015)
+        (xy -0.375024 0.250015)
+        (xy -0.375024 0.125007)
+        (xy -0.250016 0.125007)
+        (xy -0.250016 -0.125008)
+        (xy -0.125008 -0.125008)
+        (xy -0.125008 -0.625039)
+        (xy -0.250016 -0.625039)
+        (xy -0.250016 -0.750047)
+        (xy -0.500031 -0.750047)
+        (xy -0.500031 -0.625039)
+        (xy -0.625039 -0.625039)
+        (xy -0.625039 -0.500031)
+        (xy -0.875054 -0.500031)
+        (xy -0.875054 -0.875054)
+        (xy -0.750047 -0.875054)
+        (xy -0.750047 -1.000062)
+        (xy -0.625039 -1.000062)
+        (xy -0.625039 -1.12507)
+        (xy -0.375024 -1.12507)
+      ) (layer "F.SilkS") (width 0) (fill solid))
   )
   (footprint "Library:1-1437565-6" (layer "F.Cu")
